Commit message: [hw] add camera mount

File: models/rby1a/urdf/model.urdf (robot description, URDF)
Before this commit: robot RB_Y1_V1.0.1, 34 links, 33 joints
Links:
- added link rby1_camera_mount; visual mesh filename=./meshes/rby1_camera_mount_v1.obj
Joints:
- added joint head_mount: type fixed, parent link_head_2, child rby1_camera_mount, origin xyz=0.0 0.0 0.04 rpy=0.0 0.0 0.0, axis 0 0 1
